File: COMP/2021 - kicad5112 M466 Schematics/CompControl.sch (KiCad schematic (older format))
At the start: 0 parts

Commit message: The following functional blocks have been put onto their own schematic as sub-sheeets accessible through the top-sheet:             - CompControl             - DC Block             - dB Limiting and GR Buffer
	Almost all functional blocks have been wired together (Except dB Limiting/GR Buffer)

Next Steps:
	- Wire up dB Limiting/GR Buffer
	- Begin attemping simulations with Kicad's SPICE simulator.
Parts:
- added C1: 15p, M466 - Control amp:C2.5-5, symbol 2021_-_kicad5112_M466_Schematics-eagle-import:C2.5_5
- added C15: 4.7/10, M466 - Control amp:C0805, symbol 2021_-_kicad5112_M466_Schematics-eagle-import:C-USC0805
- added C2: .47/35, M466 - Control amp:C0805, symbol 2021_-_kicad5112_M466_Schematics-eagle-import:C-USC0805
- added C21: 3900p, M466-compressor-limiter:C2.5-5, symbol 2021_-_kicad5112_M466_Schematics-eagle-import:C2.5_5
- added C22: 1/35, M466-compressor-limiter:C0805, symbol 2021_-_kicad5112_M466_Schematics-eagle-import:C-USC0805
- added C23, C24: 10/25, M466-compressor-limiter:C0805, symbol 2021_-_kicad5112_M466_Schematics-eagle-import:C-USC0805
- added C26: 1/25, M466-compressor-limiter:C0805, symbol 2021_-_kicad5112_M466_Schematics-eagle-import:C-USC0805
- added C3: 1/35, M466 - Control amp:C0805, symbol 2021_-_kicad5112_M466_Schematics-eagle-import:C-USC0805
- added C4: 15P, M466 - Control amp:C2.5-5, symbol 2021_-_kicad5112_M466_Schematics-eagle-import:C2.5_5
- added C5: 3p9, M466 - Control amp:C2.5-5, symbol 2021_-_kicad5112_M466_Schematics-eagle-import:C2.5_5
- added C6: 47p, M466 - Control amp:C2.5-5, symbol 2021_-_kicad5112_M466_Schematics-eagle-import:C2.5_5
- added CR1, CR2, CR3, CR4, CR5: 1N4004, M466 - Control amp:DO41-10, symbol 2021_-_kicad5112_M466_Schematics-eagle-import:1N4004
- added CR5, CR6: 1N4004, M466-compressor-limiter:DO41-10, symbol 2021_-_kicad5112_M466_Schematics-eagle-import:1N4004
- added CR7: FLV117, M466-compressor-limiter:SMARTLED-TTW, symbol 2021_-_kicad5112_M466_Schematics-eagle-import:LED
- added IC1, Z2, Z3: LM201D, M466 - Control amp:SO08, symbol 2021_-_kicad5112_M466_Schematics-eagle-import:LM201D
- added IC4, Q1: MAT-01H, M466 - Control amp:TO78, symbol ControlAmplifier-eagle-import:MAT-01H
- added R1: 62K, M466 - Control amp:R0805, symbol Device:R_US
- added R10: 4M7, M466 - Control amp:R0805, symbol Device:R_US
- added R13: 10k, M466 - Control amp:R0805, symbol Device:R_US
- added R14, R8: 47K, M466 - Control amp:R0805, symbol Device:R_US
- added R141: 500, M466-compressor-limiter:3223G, symbol 2021_-_kicad5112_M466_Schematics-eagle-import:TRIM_US-3223G
- added R142: 620, M466-compressor-limiter:R0805, symbol Device:R_US
- added R145: 220, M466-compressor-limiter:R0805, symbol Device:R_US
- added R15: 10, M466 - Control amp:R0805, symbol Device:R_US
- added R16: 500, M466 - Control amp:3223G, symbol 2021_-_kicad5112_M466_Schematics-eagle-import:TRIM_US-3223G
- added R17: 56k, M466 - Control amp:R0805, symbol Device:R_US
- added R19, R22, R9: 620, M466 - Control amp:R0805, symbol Device:R_US
- added R2: 5K, M466 - Control amp:3223G, symbol 2021_-_kicad5112_M466_Schematics-eagle-import:TRIM_US-3223G
- added R3: 470K, M466 - Control amp:R0805, symbol Device:R_US
- added R35: 22K, M466 - Control amp:R0805, symbol Device:R_US
- added R36: 3K6, M466 - Control amp:R0805, symbol Device:R_US
- added R37: 10M, M466 - Control amp:R0805, symbol Device:R_US
- added R38: 22M, M466 - Control amp:R0805, symbol Device:R_US
- added R39: 75K, M466-compressor-limiter:R0805, symbol Device:R_US
- added R4: 15K, M466 - Control amp:R0805, symbol Device:R_US
- added R40: 3M3, M466 - Control amp:R0805, symbol Device:R_US
- added R40, R46, R47: 100K, M466-compressor-limiter:R0805, symbol Device:R_US
- added R40, R49: 5K, M466-compressor-limiter:3223G, symbol 2021_-_kicad5112_M466_Schematics-eagle-import:TRIM_US-3223G
- added R45: 7K5, M466-compressor-limiter:3223G, symbol 2021_-_kicad5112_M466_Schematics-eagle-import:TRIM_US-3223G
- added R48: 7K5, M466-compressor-limiter:R0805, symbol Device:R_US
- added R5: 220K, M466 - Control amp:R0805, symbol Device:R_US
- added R50, R51, R52: 15K, M466-compressor-limiter:R0805, symbol Device:R_US
- added R53, R54: 4K7, M466-compressor-limiter:R0805, symbol 2021_-_kicad5112_M466_Schematics-eagle-import:R-US_R0805
- added R55: 10K, M466-compressor-limiter:R0805, symbol Device:R_US
- added R57: 220K, M466-compressor-limiter:R0805, symbol Device:R_US
- added R58: 8K2, symbol Device:R_US
- added R59: 50K, M466-compressor-limiter:3223G, symbol 2021_-_kicad5112_M466_Schematics-eagle-import:TRIM_US-3223G
- added R6: 220, M466 - Control amp:R0805, symbol Device:R_US
- added R60: 4K7, M466-compressor-limiter:R0805, symbol Device:R_US
- added R84: 1k, symbol Device:R_US
- added R85: 27k, symbol Device:R_US
- added R9: 10K, M466 - Control amp:R0805, symbol Device:R_US
- added SW2A, SW2B, SW6B, SW6C: PVA2, M466-compressor-limiter:PVA2F, symbol 2021_-_kicad5112_M466_Schematics-eagle-import:PVA2
- added SW4: 8.54k, symbol Device:R_Potentiometer_US
- added SW8: R_Potentiometer_US, symbol Device:R_Potentiometer_US
- added Z6 (x2): LM201D, M466-compressor-limiter:SO08, symbol 2021_-_kicad5112_M466_Schematics-eagle-import:LM201D
Connections:
- new net: R48.1, R50.1, Z6.2 (-IN)
- new net: C23.1, R50.2, R51.1, Z6.6 (OUT)
- new net: C24.1, R52.2, Z6.6 (OUT)
- new net: C24.2, CR6.A, R54.1
- new net: R51.2, R52.1, Z6.3 (+IN)
- new net: C21.1, R47.1, R58.2, SW6B.2 (P), Z6.3 (+IN)
- new net: R48.2, R49.1 (A)
- new net: C23.2, CR5.A, R53.2
- new net: C26.1, IC1.2 (-IN), R5.1, R55.2, R57.1
- new net: R58.1, R59.1 (A), R59.2 (S)
- new net: C22.2, SW6B.1 (S)
- new net: R84.1, R85.1, SW4.3
- new net: SW2A.3 (O), SW4.2
- new net: R1.2, R2.3 (E)
- new net: R2.2 (S), R3.1
- new net: CR1.A, IC1.3 (+IN), R3.2, R38.2, R4.2, R6.1, R8.1
- new net: C2.2, R6.2
- new net: IC1.1 (ON/CMP), R9.1
- new net: C1.1, R9.2
- new net: C2.1, CR4.C, R13.1, R14.2, R141.1 (A), R142.1, R145.1, R8.2
- new net: CR2.C, R9.1
- new net: C3.1, R10.1, R46.1, R9.2, Z2.3 (+IN)
- new net: CR1.C, CR2.A, IC1.6 (OUT)
- new net: C1.2, IC1.8 (CMP)
- new net: R19.1, Z2.1 (ON/CMP)
- new net: CR3.A, R14.1, Z2.2 (-IN)
- new net: CR3.C, CR4.A, Z2.6 (OUT)
- new net: C4.1, Z2.8 (CMP)
- new net: C5.1, R22.2, Z3.1 (ON/CMP)
- new net: C5.2, CR5.C, Q1.1 (C), R13.2, R40.2, Z3.3 (+IN)
- new net: CR5.A, IC4.1 (C), R16.2 (S), R16.3 (E), Z3.6 (OUT)
- new net: C6.1, Z3.8 (CMP)
- new net: C4.2, R19.2
- new net: C6.2, R22.1
- new net: Q1.3 (E), R15.1
- new net: R15.2, R16.1 (A)
- new net: C15.1, R35.1, R40.2
- new net: R40.1, R40.2 (S)
- new net: R39.2, R40.3 (E)
- new net: R45.2 (S), R46.2
- new net: R141.2 (S), R141.3 (E), R142.2, R45.3 (E)
- new net: CR7.A@1 (A), R60.1, SW2B.2 (P)
- new net: CR5.C, CR6.C, R55.1
- new net: C21.2, C22.1, SW2A.2 (P)
- new net +15V: R37.2, R38.1, Z3.7 (V+)
- new net -16V: R1.1, R40.1
- new net AudioIn: SW4.1
- new net DCVoltageOutput: R17.2, R35.2, R36.2, R37.1
- new net Earth: R84.2, R85.2
- new net Enabled: CR7.C@1 (C), SW2B.1 (S)
- new net GND: C26.2, C3.2, R10.2, R145.2, R2.1 (A), R4.1, R40.1 (A), R45.1 (A), R47.2, R49.2 (S), R49.3 (E), R5.2, R53.1, R54.2, R57.2, Z3.2 (-IN), Z6.2 (-IN)
- new net GNDREF: SW6C.3 (O)
- new net IE14: IC4.2 (B), IC4.3 (E), R17.1, SW8.1
- new net IE15: R36.1, SW8.2
- new net VCC: R60.2
- new net bb: R59.3 (E), SW6C.2 (P)
Other:
- note added: "Bias Set"
- note added: "Bonded Together"
- note added: "Comp Control Block"
- note added: "Comp Thld Calibration"
- note added: "CompThrsHold"
- note added: "Compressor Release"
- note added: "Compressor Slope"
- note added: "Compressor Switch"
- note added: "IE1"
- note added: "IE11"
- note added: "IE2"
- note added: "IE9\n"
- note added: "Level Cal"
- note added: "OFF"
- note added: "ON"
- note added: "Output of Comp Control\n(Feed into DC Block \nbefore sending to GR Element)"
- note added: "Rel Adjustment"
- note added: "Single-Ended Audio Input"
- note added: "Slope Lin."
