File: COMP/2021 - kicad5112 M466 Schematics/LimitControl.sch (KiCad schematic (older format))
At the start: 58 parts, among them IC8 LM201D, IC9 LM201D, SW5 8.54k

Commit message: The following functional blocks have been put onto their own schematic as sub-sheeets accessible through the top-sheet:             - CompControl             - DC Block             - dB Limiting and GR Buffer
	Almost all functional blocks have been wired together (Except dB Limiting/GR Buffer)

Next Steps:
	- Wire up dB Limiting/GR Buffer
	- Begin attemping simulations with Kicad's SPICE simulator.
Parts:
- removed -VCC: VCC, symbol power:VCC
- added GND: GNDREF, symbol power:GNDREF
- CR12FLV117: value RED LED -> RED
- CR6, CR7: value 1N4004 -> 1N4148
- renumbered IC8 to Z7, IC9 to Z8
Connections:
- net GNDREF: now also S3.1 (S), GND.1 (GNDREF)
- net VCC: no longer CR12FLV117.C@1 (C), S3.1 (S)
- net IE12: now reaches C38.2, R109.1, R111.1, R27.1, Z5.3 (+IN), Z6.3 (+IN)
- net IE3: now reaches R31.2, R98.1, Z6.6 (OUT)
- net IE4: now reaches R27.2, R33.2, R98.2
- net DetectorOutput renamed DCVoltageOutput
- new net Enabled: CR12FLV117.C@1 (C), S3.1 (S)
Changed lines of the file:
@@
 $Descr User 18110 11000
 encoding utf-8
-Sheet 8 9
+Sheet 7 9
 Title "Limit Control from WBS466 Comp/Lim"
 Date "2021-05-30"
@@
 P 5450 3225
 F 0 "#GND21" H 5450 3225 50  0001 C CNN
-F 1 "GNDREF" H 5550 3175 59  0000 L BNN
+F 1 "GNDREF" H 5550 3175 59  0001 L BNN
 F 2 "" H 5450 3225 50  0001 C CNN
 F 3 "" H 5450 3225 50  0001 C CNN
@@
 $EndComp
 $Comp
-L 2021_-_kicad5112_M466_Schematics-eagle-import:LM201D IC8
+L 2021_-_kicad5112_M466_Schematics-eagle-import:LM201D Z7
 U 1 1 1433A2BB
 P 7650 2325
-F 0 "IC8" H 7550 2325 30  0000 L BNN
+F 0 "Z7" H 7550 2325 30  0000 L BNN
 F 1 "LM201D" H 7475 2250 30  0000 L BNN
 F 2 "M466-compressor-limiter:SO08" H 7650 2325 50  0001 C CNN
@@
 $EndComp
 $Comp
-L 2021_-_kicad5112_M466_Schematics-eagle-import:LM201D IC9
+L 2021_-_kicad5112_M466_Schematics-eagle-import:LM201D Z8
 U 1 1 A650351A
 P 7650 4825
-F 0 "IC9" H 7575 4850 30  0000 L BNN
+F 0 "Z8" H 7575 4850 30  0000 L BNN
 F 1 "LM201D" H 7500 4800 30  0000 L BNN
 F 2 "M466-compressor-limiter:SO08" H 7650 4825 50  0001 C CNN
@@
 U 1 1 E33CDC2D
 P 8850 4825
-F 0 "C36" H 8890 4850 59  0000 L BNN
-F 1 "10/25" H 8890 4660 59  0000 L BNN
+F 0 "C36" V 8700 4675 59  0000 L BNN
+F 1 "10/25" V 9050 4650 59  0000 L BNN
 F 2 "M466-compressor-limiter:C0805" H 8850 4825 50  0001 C CNN
 F 3 "" H 8850 4825 50  0001 C CNN
@@
 U 1 1 3633DD69
 P 9550 4825
-F 0 "CR11" H 9650 4844 59  0000 L BNN
-F 1 "1N4004" H 9650 4734 59  0000 L BNN
+F 0 "CR11" H 9625 4750 59  0000 L BNN
+F 1 "1N4004" H 9500 4900 59  0000 L BNN
 F 2 "M466-compressor-limiter:DO41-10" H 9550 4825 50  0001 C CNN
 F 3 "" H 9550 4825 50  0001 C CNN
@@
 P 4775 4050
 F 0 "CR12FLV117" H 4825 4075 59  0000 L BNN
-F 1 "RED LED" H 4825 3950 59  0000 L BNN
+F 1 "RED" H 4825 3950 59  0000 L BNN
 F 2 "M466-compressor-limiter:SMARTLED-TTW" H 4775 4050 50  0001 C CNN
 F 3 "" H 4775 4050 50  0001 C CNN
@@
 	4775 4550 4775 4725
 Connection ~ 4775 4550
-$Comp
-L power:VCC -VCC
-U 1 1 61DE52E6
-P 4775 4725
-F 0 "-VCC" H 4717 4762 50  0000 R CNN
-F 1 "VCC" H 4790 4898 50  0001 C CNN
-F 2 "" H 4775 4725 50  0001 C CNN
-F 3 "" H 4775 4725 50  0001 C CNN
-	1    4775 4725
-	-1   0    0    1
-$EndComp
 Wire Wire Line
 	5450 2425 7350 2425
@@
 AR Path="/62CD61A4/621EBECA" Ref="CR6"  Part="1"
 F 0 "CR6" H 14250 3350 59  0000 L BNN
-F 1 "1N4004" H 14250 3500 59  0000 L BNN
+F 1 "1N4148" H 14250 3500 59  0000 L BNN
 F 2 "M466 - Control amp:DO41-10" H 14500 3425 50  0001 C CNN
 F 3 "" H 14500 3425 50  0001 C CNN
@@
 AR Path="/62CD61A4/621EBED0" Ref="CR7"  Part="1"
 F 0 "CR7" H 14250 3950 59  0000 L BNN
-F 1 "1N4004" H 14075 3800 59  0000 L BNN
+F 1 "1N4148" H 14075 3800 59  0000 L BNN
 F 2 "M466 - Control amp:DO41-10" H 14200 3925 50  0001 C CNN
 F 3 "" H 14200 3925 50  0001 C CNN
@@
 AR Path="/60CA7A69/621EC086" Ref="R?"  Part="1"
 AR Path="/621EC086" Ref="R35"  Part="1"
-AR Path="/62CD61A4/621EC086" Ref="R35"  Part="1"
-F 0 "R35" H 12150 4150 59  0000 L BNN
+AR Path="/62CD61A4/621EC086" Ref="R25"  Part="1"
+F 0 "R25" H 12150 4150 59  0000 L BNN
 F 1 "5K" H 12200 4050 59  0000 L BNN
 F 2 "M466 - Control amp:3223G" H 12400 4125 50  0001 C CNN
@@
 AR Path="/621EC0B6" Ref="R29"  Part="1"
 AR Path="/62CD61A4/621EC0B6" Ref="R29"  Part="1"
-F 0 "R29" V 12925 6350 59  0000 L BNN
-F 1 "51K" V 12825 6275 59  0000 L BNN
+F 0 "R29" V 13125 6250 59  0000 L BNN
+F 1 "51K" V 12925 6250 59  0000 L BNN
 F 2 "M466 - Control amp:R0805" H 13000 6325 50  0001 C CNN
 F 3 "" H 13000 6325 50  0001 C CNN
@@
 AR Path="/621EC0C2" Ref="R31"  Part="1"
 AR Path="/62CD61A4/621EC0C2" Ref="R31"  Part="1"
-F 0 "R31" V 13725 6725 59  0000 L BNN
-F 1 "22K" V 13625 6675 59  0000 L BNN
+F 0 "R31" V 13925 6650 59  0000 L BNN
+F 1 "22K" V 13725 6650 59  0000 L BNN
 F 2 "M466 - Control amp:R0805" H 13800 6725 50  0001 C CNN
 F 3 "" H 13800 6725 50  0001 C CNN
@@
 P 15175 7300
 F 0 "#PWR?" H 15175 7050 50  0001 C CNN
-F 1 "GNDREF" H 15180 7127 50  0000 C CNN
+F 1 "GNDREF" H 15180 7127 50  0001 C CNN
 F 2 "" H 15175 7300 50  0001 C CNN
 F 3 "" H 15175 7300 50  0001 C CNN
@@
 	13500 2525 13500 3425
 $Comp
-L power:GNDREF #GND38
+L power:GNDREF GND
 U 1 1 2DA03382
 P 3575 4350
-F 0 "#GND38" H 3575 4350 50  0001 C CNN
-F 1 "GNDREF" H 3475 4250 59  0000 L BNN
+F 0 "GND" H 3575 4350 50  0001 C CNN
+F 1 "GNDREF" H 3475 4250 59  0001 L BNN
 F 2 "" H 3575 4350 50  0001 C CNN
 F 3 "" H 3575 4350 50  0001 C CNN
@@
 AR Path="/621EC0E0" Ref="R39"  Part="1"
 AR Path="/62CD61A4/621EC0E0" Ref="R39"  Part="1"
-F 0 "R39" V 12925 5925 59  0000 L BNN
-F 1 "1M" V 12825 5875 59  0000 L BNN
+F 0 "R39" V 13125 5900 59  0000 L BNN
+F 1 "1M" V 12950 5900 59  0000 L BNN
 F 2 "M466 - Control amp:R0805" H 13000 5925 50  0001 C CNN
 F 3 "" H 13000 5925 50  0001 C CNN
@@
 	14400 4525 14650 4525
 Text HLabel 16300 3500 2    50   Output ~ 0
-DetectorOutput
+DCVoltageOutput
 Text Notes 16300 4375 0    50   ~ 0
 (Feed into GR/Limit LEDs Block)
@@
 Wire Wire Line
 	950  4175 2800 4175
+Wire Wire Line
+	3575 4350 3575 4250
+Text Label 11750 2325 0    50   ~ 0
+IE12
+Text Label 14600 5825 0    50   ~ 0
+IE3
+Text Label 14925 6475 0    50   ~ 0
+IE4
+Text HLabel 4775 4725 2    50   BiDi ~ 0
+Enabled
 $EndSCHEMATC
