File: COMP/2021 - kicad5112 M466 Schematics/OutputAmplifier.sch (KiCad schematic (older format))
At the start: 73 parts, among them IC1 LM201D, IC2 LM201D, Q1 NPN-TRANSISTOR_SOT23, Q2 PNP-TRANSISTOR_SOT23, Q3 NPN-TRANSISTOR_SOT23, Q4 PNP-TRANSISTOR_SOT23, Q5 NPN-TRANSISTOR_SOT23, Q6 PNP-TRANSISTOR_SOT23, Q7 NPN-TRANSISTOR_SOT23, Q8 PNP-TRANSISTOR_SOT23

Commit message: The following functional blocks have been put onto their own schematic as sub-sheeets accessible through the top-sheet:             - CompControl             - DC Block             - dB Limiting and GR Buffer
	Almost all functional blocks have been wired together (Except dB Limiting/GR Buffer)

Next Steps:
	- Wire up dB Limiting/GR Buffer
	- Begin attemping simulations with Kicad's SPICE simulator.
Parts:
- removed E1, E2, E3, E4, E5, E6, E7: SMD2, OutputAmplifier:SMD1,27-2,54, symbol OutputAmplifier-eagle-import:SMD2
Connections:
- net E2: now reaches C2.2, R2.1
- net E3: now reaches Q3.3 (C), R13.2, R17.2, R19.1
- net E1: now reaches C1.2, R1.2
- net E4: now reaches C15.1, R36.1
- net E7: now reaches Q8.3 (C), R14.2, R29.2
- net E6: now reaches C16.1, R37.2
- net GND renamed E5
Changed lines of the file:
@@
 $Descr A2 23386 16535
 encoding utf-8
-Sheet 1 9
+Sheet 2 9
 Title "M466 Output Amplifier"
 Date "2021-11-27"
@@
 $EndComp
 $Comp
-L OutputAmplifier-eagle-import:SMD2 E1
-U 1 1 EF75A04C
-P 5175 3975
-F 0 "E1" H 5130 4048 59  0000 L BNN
-F 1 "SMD2" H 5130 3845 59  0000 L BNN
-F 2 "OutputAmplifier:SMD1,27-2,54" H 5175 3975 50  0001 C CNN
-F 3 "" H 5175 3975 50  0001 C CNN
-	1    5175 3975
-	1    0    0    -1
-$EndComp
-$Comp
-L OutputAmplifier-eagle-import:SMD2 E2
-U 1 1 12AD0590
-P 5075 9875
-F 0 "E2" H 5030 9948 59  0000 L BNN
-F 1 "SMD2" H 5030 9745 59  0000 L BNN
-F 2 "OutputAmplifier:SMD1,27-2,54" H 5075 9875 50  0001 C CNN
-F 3 "" H 5075 9875 50  0001 C CNN
-	1    5075 9875
-	1    0    0    -1
-$EndComp
-$Comp
 L OutputAmplifier-eagle-import:C2.5_5 C17
 U 1 1 23CE9F0E
@@
 $EndComp
 $Comp
-L OutputAmplifier-eagle-import:SMD2 E3
-U 1 1 0146C692
-P 16075 2675
-F 0 "E3" H 16030 2748 59  0000 L BNN
-F 1 "SMD2" H 16030 2545 59  0000 L BNN
-F 2 "OutputAmplifier:SMD1,27-2,54" H 16075 2675 50  0001 C CNN
-F 3 "" H 16075 2675 50  0001 C CNN
-	1    16075 2675
-	-1   0    0    1
-$EndComp
-$Comp
-L OutputAmplifier-eagle-import:SMD2 E4
-U 1 1 E410CEFF
-P 16075 4675
-F 0 "E4" H 16030 4748 59  0000 L BNN
-F 1 "SMD2" H 16030 4545 59  0000 L BNN
-F 2 "OutputAmplifier:SMD1,27-2,54" H 16075 4675 50  0001 C CNN
-F 3 "" H 16075 4675 50  0001 C CNN
-	1    16075 4675
-	-1   0    0    1
-$EndComp
-$Comp
-L OutputAmplifier-eagle-import:SMD2 E5
-U 1 1 557D9ADD
-P 15975 7875
-F 0 "E5" H 15930 7948 59  0000 L BNN
-F 1 "SMD2" H 15930 7745 59  0000 L BNN
-F 2 "OutputAmplifier:SMD1,27-2,54" H 15975 7875 50  0001 C CNN
-F 3 "" H 15975 7875 50  0001 C CNN
-	1    15975 7875
-	-1   0    0    1
-$EndComp
-$Comp
-L OutputAmplifier-eagle-import:SMD2 E6
-U 1 1 BB2A911A
-P 15975 10375
-F 0 "E6" H 15930 10448 59  0000 L BNN
-F 1 "SMD2" H 15930 10245 59  0000 L BNN
-F 2 "OutputAmplifier:SMD1,27-2,54" H 15975 10375 50  0001 C CNN
-F 3 "" H 15975 10375 50  0001 C CNN
-	1    15975 10375
-	-1   0    0    1
-$EndComp
-$Comp
-L OutputAmplifier-eagle-import:SMD2 E7
-U 1 1 05F8F254
-P 15975 13275
-F 0 "E7" H 15930 13348 59  0000 L BNN
-F 1 "SMD2" H 15930 13145 59  0000 L BNN
-F 2 "OutputAmplifier:SMD1,27-2,54" H 15975 13275 50  0001 C CNN
-F 3 "" H 15975 13275 50  0001 C CNN
-	1    15975 13275
-	-1   0    0    1
-$EndComp
-$Comp
 L OutputAmplifier-eagle-import:GND #SUPPLY6
 U 1 1 137BDED3
@@
 	1    0    0    -1
 $EndComp
+Text HLabel 5275 3975 0    50   Input ~ 0
+E1
+Text HLabel 5175 9875 0    50   Input ~ 0
+E2
+Text HLabel 15875 13275 2    50   BiDi ~ 0
+E7
+Text HLabel 15875 10375 2    50   BiDi ~ 0
+E6
+Text HLabel 15875 7875 2    50   BiDi ~ 0
+E5
+Text HLabel 15975 4675 2    50   BiDi ~ 0
+E4
+Text HLabel 15975 2675 2    50   Input ~ 0
+E3
 $EndSCHEMATC
