File: COMP/2021 - kicad5112 M466 Schematics/2021 - kicad5112 M466 Schematics.sch (KiCad schematic (older format))
At the start: 231 parts, among them IC1 LM201D, IC10 LM201D, IC11 LM201D, IC12 LM201D, IC13 LM201D, IC2 LM201D, IC3 LM201D, IC4 LM201D, IC5 LM201D, IC6 LM201D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

Commit message: The following functional blocks have been put onto their own schematic as sub-sheeets accessible through the top-sheet: 	- BST 	- GR Element 	- BUF (VU)
Parts:
- removed C10, C12: 220p, 2021 - kicad5112 M466 Schematics:C2.5-5, symbol 2021_-_kicad5112_M466_Schematics-eagle-import:C2.5_5
- removed C11, C13: 4p7, 2021 - kicad5112 M466 Schematics:C2.5-5, symbol 2021_-_kicad5112_M466_Schematics-eagle-import:C2.5_5
- removed C14, C15, C31, C8, C9: 33/10, 2021 - kicad5112 M466 Schematics:C0805, symbol 2021_-_kicad5112_M466_Schematics-eagle-import:C-USC0805
- removed C16: 6p8, 2021 - kicad5112 M466 Schematics:C2.5-5, symbol 2021_-_kicad5112_M466_Schematics-eagle-import:C2.5_5
- removed C17: 15p, 2021 - kicad5112 M466 Schematics:C2.5-5, symbol 2021_-_kicad5112_M466_Schematics-eagle-import:C2.5_5
- removed C18, C41: 10/25, 2021 - kicad5112 M466 Schematics:C0805, symbol 2021_-_kicad5112_M466_Schematics-eagle-import:C-USC0805
- removed C19: 22p, 2021 - kicad5112 M466 Schematics:C2.5-5, symbol 2021_-_kicad5112_M466_Schematics-eagle-import:C2.5_5
- removed C20: 150/6, 2021 - kicad5112 M466 Schematics:C0805, symbol 2021_-_kicad5112_M466_Schematics-eagle-import:C-USC0805
- removed C27: 47p, 2021 - kicad5112 M466 Schematics:C2.5-5, symbol 2021_-_kicad5112_M466_Schematics-eagle-import:C2.5_5
- removed C28: 8p2, 2021 - kicad5112 M466 Schematics:C2.5-5, symbol 2021_-_kicad5112_M466_Schematics-eagle-import:C2.5_5
- removed C29: 2p7, 2021 - kicad5112 M466 Schematics:C2.5-5, symbol 2021_-_kicad5112_M466_Schematics-eagle-import:C2.5_5
- removed C30: 330/6, 2021 - kicad5112 M466 Schematics:C0805, symbol 2021_-_kicad5112_M466_Schematics-eagle-import:C-USC0805
- removed CR8, CR9: 1N4004, 2021 - kicad5112 M466 Schematics:DO41-10, symbol 2021_-_kicad5112_M466_Schematics-eagle-import:1N4004
- removed IC1, IC13, IC2, IC3, IC4, IC5: LM201D, 2021 - kicad5112 M466 Schematics:SO08, symbol 2021_-_kicad5112_M466_Schematics-eagle-import:LM201D
- removed INPUT1, INPUT2: SMD2, 2021 - kicad5112 M466 Schematics:SMD1,27-2,54, symbol 2021_-_kicad5112_M466_Schematics-eagle-import:SMD2
- removed Q4: MAT-04D, 2021 - kicad5112 M466 Schematics:SO14, symbol 2021_-_kicad5112_M466_Schematics-eagle-import:MAT-04D
- removed R13, R14: 75K, 2021 - kicad5112 M466 Schematics:R0805, symbol 2021_-_kicad5112_M466_Schematics-eagle-import:R-US_R0805
- removed R132: 20K, 2021 - kicad5112 M466 Schematics:3223G, symbol 2021_-_kicad5112_M466_Schematics-eagle-import:TRIM_US-3223G
- removed R133: 10K, 2021 - kicad5112 M466 Schematics:R0805, symbol 2021_-_kicad5112_M466_Schematics-eagle-import:R-US_R0805
- removed R134: 300K, 2021 - kicad5112 M466 Schematics:R0805, symbol 2021_-_kicad5112_M466_Schematics-eagle-import:R-US_R0805
- removed R135: 3K9, 2021 - kicad5112 M466 Schematics:R0805, symbol 2021_-_kicad5112_M466_Schematics-eagle-import:R-US_R0805
- removed R137: 3K3, 2021 - kicad5112 M466 Schematics:R0805, symbol 2021_-_kicad5112_M466_Schematics-eagle-import:R-US_R0805
- removed R15, R32: 15k, 2021 - kicad5112 M466 Schematics:R0805, symbol 2021_-_kicad5112_M466_Schematics-eagle-import:R-US_R0805
- removed R16, R17, R19: 15K, 2021 - kicad5112 M466 Schematics:R0805, symbol 2021_-_kicad5112_M466_Schematics-eagle-import:R-US_R0805
- removed R18, R20, R62: 620, 2021 - kicad5112 M466 Schematics:R0805, symbol 2021_-_kicad5112_M466_Schematics-eagle-import:R-US_R0805
- removed R21: 47K, 2021 - kicad5112 M466 Schematics:R0805, symbol 2021_-_kicad5112_M466_Schematics-eagle-import:R-US_R0805
- removed R22: 3K6, 2021 - kicad5112 M466 Schematics:R0805, symbol 2021_-_kicad5112_M466_Schematics-eagle-import:R-US_R0805
- removed R23: 22K, 2021 - kicad5112 M466 Schematics:R0805, symbol 2021_-_kicad5112_M466_Schematics-eagle-import:R-US_R0805
- removed R27, R63: 150K, 2021 - kicad5112 M466 Schematics:R0805, symbol 2021_-_kicad5112_M466_Schematics-eagle-import:R-US_R0805
- removed R28: 1k, 2021 - kicad5112 M466 Schematics:R0805, symbol 2021_-_kicad5112_M466_Schematics-eagle-import:R-US_R0805
- removed R29: 15p, 2021 - kicad5112 M466 Schematics:R0805, symbol 2021_-_kicad5112_M466_Schematics-eagle-import:R-US_R0805
- removed R30: 1K, 2021 - kicad5112 M466 Schematics:R0805, symbol 2021_-_kicad5112_M466_Schematics-eagle-import:R-US_R0805
- removed R31: 2K2, 2021 - kicad5112 M466 Schematics:R0805, symbol 2021_-_kicad5112_M466_Schematics-eagle-import:R-US_R0805
- removed R34: 470, 2021 - kicad5112 M466 Schematics:R0805, symbol 2021_-_kicad5112_M466_Schematics-eagle-import:R-US_R0805
- removed R35: 500, 2021 - kicad5112 M466 Schematics:3223G, symbol 2021_-_kicad5112_M466_Schematics-eagle-import:TRIM_US-3223G
- removed R61: 75, 2021 - kicad5112 M466 Schematics:R0805, symbol 2021_-_kicad5112_M466_Schematics-eagle-import:R-US_R0805
- removed R64, R65: 100K, 2021 - kicad5112 M466 Schematics:R0805, symbol 2021_-_kicad5112_M466_Schematics-eagle-import:R-US_R0805
- removed R66, R67: 1M, 2021 - kicad5112 M466 Schematics:R0805, symbol 2021_-_kicad5112_M466_Schematics-eagle-import:R-US_R0805
- removed R68: 5K, 2021 - kicad5112 M466 Schematics:R0805, symbol 2021_-_kicad5112_M466_Schematics-eagle-import:R-US_R0805
- removed R69, R71: 33K, 2021 - kicad5112 M466 Schematics:R0805, symbol 2021_-_kicad5112_M466_Schematics-eagle-import:R-US_R0805
- removed R70: 5K, 2021 - kicad5112 M466 Schematics:3223G, symbol 2021_-_kicad5112_M466_Schematics-eagle-import:TRIM_US-3223G
- removed T14: 2N2222, 2021 - kicad5112 M466 Schematics:TO92-EBC-OVAL, symbol 2021_-_kicad5112_M466_Schematics-eagle-import:2N2222
- renumbered S6 to SW9A, S5 to SW9B
Connections:
- wire segments 625 -> 434
Other:
- note added: "Compressor ON"
- note added: "GR/VU switch"
- note added: "Make-up \nGain"

Commit message: Limit Control Block schematic imported fully into its own sheet (LimitControl.sch)
Connections:
- wire segments 434 -> 437
Other:
- note added: "BUF"
- note added: "GR"
- note added: "VU"
- moved on the sheet: -COM, -COM1, -COM10, -COM5, -COM6, C1, C2, C3, C4, C43, C5, C6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

Commit message: The following functional blocks have been put onto their own schematic as sub-sheeets accessible through the top-sheet:             - CompControl             - DC Block             - dB Limiting and GR Buffer
	Almost all functional blocks have been wired together (Except dB Limiting/GR Buffer)

Next Steps:
	- Wire up dB Limiting/GR Buffer
	- Begin attemping simulations with Kicad's SPICE simulator.
Parts:
- removed 2E1, 2E2, 2E3, 2E4, 2E5, 2E6, 2E7, IE1, IE10, IE15, IE2, IE9, IR141, UNK15, UNK16: SMD2, 2021 - kicad5112 M466 Schematics:SMD1,27-2,54, symbol 2021_-_kicad5112_M466_Schematics-eagle-import:SMD2
- removed C21, C23, C24: 10/25, 2021 - kicad5112 M466 Schematics:C0805, symbol 2021_-_kicad5112_M466_Schematics-eagle-import:C-USC0805
- removed C22: 0.022, 2021 - kicad5112 M466 Schematics:C2.5-5, symbol 2021_-_kicad5112_M466_Schematics-eagle-import:C2.5_5
- removed C26: 1/25, 2021 - kicad5112 M466 Schematics:C0805, symbol 2021_-_kicad5112_M466_Schematics-eagle-import:C-USC0805
- removed CR5, CR6: 1N4004, 2021 - kicad5112 M466 Schematics:DO41-10, symbol 2021_-_kicad5112_M466_Schematics-eagle-import:1N4004
- removed IC6, IC7: LM201D, 2021 - kicad5112 M466 Schematics:SO08, symbol 2021_-_kicad5112_M466_Schematics-eagle-import:LM201D
- removed LED3, LED4, LED5: LED, 2021 - kicad5112 M466 Schematics:SMARTLED-TTW, symbol 2021_-_kicad5112_M466_Schematics-eagle-import:LED
- removed R112, R53, R54, R60: 4K7, 2021 - kicad5112 M466 Schematics:R0805, symbol 2021_-_kicad5112_M466_Schematics-eagle-import:R-US_R0805
- removed R131, R55: 10K, 2021 - kicad5112 M466 Schematics:R0805, symbol 2021_-_kicad5112_M466_Schematics-eagle-import:R-US_R0805
- removed R136: 5K1, 2021 - kicad5112 M466 Schematics:R0805, symbol 2021_-_kicad5112_M466_Schematics-eagle-import:R-US_R0805
- removed R141: 500, 2021 - kicad5112 M466 Schematics:R0805, symbol 2021_-_kicad5112_M466_Schematics-eagle-import:R-US_R0805
- removed R142: 620, 2021 - kicad5112 M466 Schematics:R0805, symbol 2021_-_kicad5112_M466_Schematics-eagle-import:R-US_R0805
- removed R145: 220, 2021 - kicad5112 M466 Schematics:R0805, symbol 2021_-_kicad5112_M466_Schematics-eagle-import:R-US_R0805
- removed R33, R41, R43, R46, R47: 100K, 2021 - kicad5112 M466 Schematics:R0805, symbol 2021_-_kicad5112_M466_Schematics-eagle-import:R-US_R0805
- removed R39: 75K, 2021 - kicad5112 M466 Schematics:R0805, symbol 2021_-_kicad5112_M466_Schematics-eagle-import:R-US_R0805
- removed R40, R49: 5K, 2021 - kicad5112 M466 Schematics:3223G, symbol 2021_-_kicad5112_M466_Schematics-eagle-import:TRIM_US-3223G
- removed R45: 7K5, 2021 - kicad5112 M466 Schematics:3223G, symbol 2021_-_kicad5112_M466_Schematics-eagle-import:TRIM_US-3223G
- removed R48: 7K5, 2021 - kicad5112 M466 Schematics:R0805, symbol 2021_-_kicad5112_M466_Schematics-eagle-import:R-US_R0805
- removed R50, R51, R52: 15K, 2021 - kicad5112 M466 Schematics:R0805, symbol 2021_-_kicad5112_M466_Schematics-eagle-import:R-US_R0805
- removed R58: 8K2, 2021 - kicad5112 M466 Schematics:R0805, symbol 2021_-_kicad5112_M466_Schematics-eagle-import:R-US_R0805
- removed R59: 50K, 2021 - kicad5112 M466 Schematics:3223G, symbol 2021_-_kicad5112_M466_Schematics-eagle-import:TRIM_US-3223G
- removed S1: 3PDT, 2021 - kicad5112 M466 Schematics:3PDT, symbol 2021_-_kicad5112_M466_Schematics-eagle-import:3PDT
- removed S2, S3: PVA2, 2021 - kicad5112 M466 Schematics:PVA2F, symbol 2021_-_kicad5112_M466_Schematics-eagle-import:PVA2
- added C42: 47/40, symbol Device:C_Polarized_US
- added GND (x2), GND?: GNDREF, symbol power:GNDREF
- added R131: 10K, symbol Device:R_US
- added SW1B: 31k, symbol Device:R_Potentiometer_US
- renumbered S4 to SW2C, S7 to SW7C
Connections:
- net labels added: +24V, -24V, pin15, pin16, v, w
- wire segments 437 -> 329
Other:
- note added: "Insert"
- note added: "OUTPUT AMPLFIER\n4-109D"
- note added: "Output\n"
- note added: "Sensitivity"
- note added: "Switches Tied\nSW2A, SW2B and SW2C"
- note added: "VU BUF"
- note removed: "BUF"
- note removed: "DSFSDF"
- note removed: "OUTPUT AMPLFIER"
- moved on the sheet: R72, R73, SW2C

Commit message: Orignal M466 Schematic has been fully split and wired up into sub-schematic sheets corresponding to functional blocks.
Next steps:
	- Verify through simulation
Parts:
- removed C32: 100p, 2021 - kicad5112 M466 Schematics:C2.5-5, symbol 2021_-_kicad5112_M466_Schematics-eagle-import:C2.5_5
- removed C33: 3p9, 2021 - kicad5112 M466 Schematics:C2.5-5, symbol 2021_-_kicad5112_M466_Schematics-eagle-import:C2.5_5
- removed C34: 8p2, 2021 - kicad5112 M466 Schematics:C2.5-5, symbol 2021_-_kicad5112_M466_Schematics-eagle-import:C2.5_5
- removed C35, C36: 10/25, 2021 - kicad5112 M466 Schematics:C0805, symbol 2021_-_kicad5112_M466_Schematics-eagle-import:C-USC0805
- removed C38: 1/35, 2021 - kicad5112 M466 Schematics:C0805, symbol 2021_-_kicad5112_M466_Schematics-eagle-import:C-USC0805
- removed C39, C40: 22/25, 2021 - kicad5112 M466 Schematics:C0805, symbol 2021_-_kicad5112_M466_Schematics-eagle-import:C-USC0805
- removed CR10, CR11, CR13, CR14: 1N4004, 2021 - kicad5112 M466 Schematics:DO41-10, symbol 2021_-_kicad5112_M466_Schematics-eagle-import:1N4004
- removed IC10, IC11, IC12, IC8, IC9: LM201D, 2021 - kicad5112 M466 Schematics:SO08, symbol 2021_-_kicad5112_M466_Schematics-eagle-import:LM201D
- removed IE11, IE12, IE13, IE3, IE4, IE5, IE6, IE7: SMD2, 2021 - kicad5112 M466 Schematics:SMD1,27-2,54, symbol 2021_-_kicad5112_M466_Schematics-eagle-import:SMD2
- removed LED1, LED2: LED, 2021 - kicad5112 M466 Schematics:SMARTLED-TTW, symbol 2021_-_kicad5112_M466_Schematics-eagle-import:LED
- removed R100, R107, R108: 4K7, 2021 - kicad5112 M466 Schematics:R0805, symbol 2021_-_kicad5112_M466_Schematics-eagle-import:R-US_R0805
- removed R101: 20K, 2021 - kicad5112 M466 Schematics:3223G, symbol 2021_-_kicad5112_M466_Schematics-eagle-import:TRIM_US-3223G
- removed R102, R105, R124, R125: 620, 2021 - kicad5112 M466 Schematics:R0805, symbol 2021_-_kicad5112_M466_Schematics-eagle-import:R-US_R0805
- removed R103, R120, R99: 100K, 2021 - kicad5112 M466 Schematics:R0805, symbol 2021_-_kicad5112_M466_Schematics-eagle-import:R-US_R0805
- removed R104, R106: 15K, 2021 - kicad5112 M466 Schematics:R0805, symbol 2021_-_kicad5112_M466_Schematics-eagle-import:R-US_R0805
- removed R109: 1K, 2021 - kicad5112 M466 Schematics:R0805, symbol 2021_-_kicad5112_M466_Schematics-eagle-import:R-US_R0805
- removed R111, R117: 10M, 2021 - kicad5112 M466 Schematics:R0805, symbol 2021_-_kicad5112_M466_Schematics-eagle-import:R-US_R0805
- removed R113: 1M, 2021 - kicad5112 M466 Schematics:R0805, symbol 2021_-_kicad5112_M466_Schematics-eagle-import:R-US_R0805
- removed R114, R115: 510, 2021 - kicad5112 M466 Schematics:R0805, symbol 2021_-_kicad5112_M466_Schematics-eagle-import:R-US_R0805
- removed R116: 5K1, 2021 - kicad5112 M466 Schematics:R0805, symbol 2021_-_kicad5112_M466_Schematics-eagle-import:R-US_R0805
- removed R118: 75K, 2021 - kicad5112 M466 Schematics:R0805, symbol 2021_-_kicad5112_M466_Schematics-eagle-import:R-US_R0805
- removed R119: 5K, 2021 - kicad5112 M466 Schematics:3223G, symbol 2021_-_kicad5112_M466_Schematics-eagle-import:TRIM_US-3223G
- removed R121, R122, R139: 47K, 2021 - kicad5112 M466 Schematics:R0805, symbol 2021_-_kicad5112_M466_Schematics-eagle-import:R-US_R0805
- removed R123: 120K, 2021 - kicad5112 M466 Schematics:R0805, symbol 2021_-_kicad5112_M466_Schematics-eagle-import:R-US_R0805
- removed R126, R127: 2K7, 2021 - kicad5112 M466 Schematics:R0805, symbol 2021_-_kicad5112_M466_Schematics-eagle-import:R-US_R0805
- removed R57: 220K, 2021 - kicad5112 M466 Schematics:R0805, symbol 2021_-_kicad5112_M466_Schematics-eagle-import:R-US_R0805
- removed R98: 7K5, 2021 - kicad5112 M466 Schematics:3223G, symbol 2021_-_kicad5112_M466_Schematics-eagle-import:TRIM_US-3223G
Connections:
- net dBLimLEDs_GRBUF/OutputGRVUMeter: now also SW9A.3 (S)
Other:
- note removed: "CONTROL AMPLIFIER"
- moved on the sheet: -COM, -COM1, -COM10, -COM5, -COM6, C1, C2, C3, C4, C42, C43, C44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
